File: schematics/DEVI/Devi.sch (EAGLE design)
At the start: 124 parts

Commit message: latest
Other:
- note added: "RED - 1k GREEN - 4k7 BLUE - 680 Ohm"
Changed lines of the file:
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@@
 <setting verticaltext="up"/>
 </settings>
-<grid distance="0.1" unitdist="inch" unit="inch" style="lines" multiple="1" display="yes" altdistance="0.01" altunitdist="inch" altunit="inch"/>
+<grid distance="0.1" unitdist="inch" unit="inch" style="lines" multiple="1" display="no" altdistance="0.01" altunitdist="inch" altunit="inch"/>
 <layers>
 <layer number="1" name="Top" color="4" fill="1" visible="no" active="no"/>
@@
 <text x="272.288" y="145.288" size="1.778" layer="94">*</text>
 <text x="282.702" y="141.732" size="1.778" layer="94">* - This should be used for an analog low pass filter</text>
+<text x="38.1" y="129.54" size="1.778" layer="91">RED - 1k
+GREEN - 4k7
+BLUE - 680 Ohm</text>
 </plain>
 <instances>
