File: schematics/DEVI Lite/Devi_Lite.brd (EAGLE design)
At the start: 99.7 x 56.2 mm, 96 parts

Commit message: latest
Parts:
- moved R7 17.8 mm to (91.4, 189.2)
- moved SW7 17.8 mm to (81.3, 189.2)
- moved LED7 10.2 mm to (71.1, 201.9)
- moved R15 2.54 mm to (41.9, 215.9)
- moved R19 2.01 mm to (47.6, 179.7)
- moved R20 1.42 mm to (42.5, 176.5)
- moved R9 1.27 mm to (36.8, 174.0)
Connections:
- removed net N$10: R17.P$1, S1.9
- removed net N$11: R18.P$1, S1.10
- removed net N$12: R19.P$1, S1.11
- removed net N$13: R20.P$1, S1.12
- removed net N$2: R9.P$1, S1.1
- removed net N$3: R10.P$1, S1.2
- removed net N$4: R11.P$1, S1.3
- removed net N$5: R12.P$1, S1.4
- removed net N$6: R13.P$1, S1.5
- removed net N$7: R14.P$1, S1.6
- removed net N$8: R15.P$1, S1.7
- removed net N$9: R16.P$1, S1.8
- net +5V: now also S1.A
- net GND: now also R10.P$2, R11.P$2, R12.P$2, R13.P$2, R14.P$2, R15.P$2, R16.P$2, R17.P$2, R18.P$2, R19.P$2, R20.P$2, R9.P$2; no longer S1.A
- net JS1: now also R9.P$1, S1.1; no longer R9.P$2
- net JS10: now also R18.P$1, S1.10; no longer R18.P$2
- net JS11: now also R19.P$1, S1.11; no longer R19.P$2
- net JS12: now also R20.P$1, S1.12; no longer R20.P$2
- net JS2: now also R10.P$1, S1.2; no longer R10.P$2
- net JS3: now also R11.P$1, S1.3; no longer R11.P$2
- net JS4: now also R12.P$1, S1.4; no longer R12.P$2
- net JS5: now also R13.P$1, S1.5; no longer R13.P$2
- net JS6: now also R14.P$1, S1.6; no longer R14.P$2
- net JS7: now also R15.P$1, S1.7; no longer R15.P$2
- net JS8: now also R16.P$1, S1.8; no longer R16.P$2
- net JS9: now also R17.P$1, S1.9; no longer R17.P$2
Routing:
- net JS10: track 160.1 -> 21.5 mm
- net JS11: track 141.7 -> 18.1 mm
- net JS12: track 124.4 -> 17.8 mm
- net JS1: track 106.9 -> 20.3 mm
- net JS2: track 90.3 -> 24.4 mm
- net GND: track 1008.9 -> 1064.6 mm
- net JS3: track 79.2 -> 26.8 mm
- net JB7: track 355.0 -> 371.2 mm
- net +5V: track 866.3 -> 855.3 mm
- net JS4: track 36.8 -> 27.2 mm
- net JS7: track 15.9 -> 25.1 mm
- net JS9: track 14.0 -> 23.0 mm
- net N$4: track 8.02 -> 0.00 mm
- net JS8: track 13.3 -> 19.7 mm
- net N$11: track 6.27 -> 0.00 mm
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Other:
- board text added: "1"
- board text added: "10"
- board text added: "2"
- board text added: "20"
- board text added: "3"
- board text added: "30"
- board text added: "4"
- board text added: "5"
- board text added: "6"
- board text added: "7"
- board text added: "8"
- board text added: "9"
- board text added: "A"
- board text added: "B"
- board text added: "C"
- board text added: "D"
- board text added: "E"
- board text added: "F"
- board text added: "G"
- board text added: "H"
- board text added: "I"
- board text added: "J"
- board text added: "JP8-2"
- board text added: "JP8-3"
- board text added: "K"
- board text added: "L"
- board text added: "M"
- board text added: "N"
- board text added: "O"
- board text added: "P"
- board text added: "Q"
- board text added: "R"
- board text added: "S"
- board text added: "T"
- board text added: "U"
- board text added: "V"
- board text removed: "LE"
